File: tinyPEPPER2.kicad_pcb (KiCad board)
At the start: 4 copper layers, 20 x 20 mm, 163 parts, among them T201 BC847, T202 BC847, T203 BC847, T301 BC847, T302 BC847, T303 BC847, T401 BC847, T402 BC847, T403 BC847, T501 BC847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

Commit message: got it working in kicad7
Other:
- net class 8mil removed
- net class Default removed
- net class SUPPLY removed
