File: single_esc_update.kicad_sch (KiCad schematic)
At the start: 44 parts, among them J1 Conn_01x03, Q1 BC847, Q2 PMOS, Q3 NMOS, Q4 BC847, Q5 NMOS, Q6 PMOS, Q7 BC847, Q8 NMOS, Q9 PMOS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

Commit message: forget
Parts:
- removed JP1: Jumper, symbol Jumper:SolderJumper_2_Open
- added C9: 22µF, Capacitor_SMD:C_0805_2012Metric, symbol Device:C_Small
- added FB1: Ferrite, Inductor_SMD:L_0402_1005Metric, symbol Device:FerriteBead_Small
- added J2: Conn_01x03, Connector_PinHeader_2.54mm:PinHeader_1x03_P2.54mm_Vertical, symbol Connector_Generic:Conn_01x03
- added TP1, TP4: vcc, TestPoint:TestPoint_Pad_3.0x3.0mm, symbol Connector:TestPoint_Small
- added TP10: 3,3v, TestPoint:TestPoint_Pad_D1.0mm, symbol Connector:TestPoint_Small
- added TP2: gnd, TestPoint:TestPoint_Pad_3.0x3.0mm, symbol Connector:TestPoint_Small
- added TP3: p0,5, TestPoint:TestPoint_Pad_D1.0mm, symbol Connector:TestPoint_Small
- added TP8: rst, TestPoint:TestPoint_Pad_D1.0mm, symbol Connector:TestPoint_Small
- added TP9: gnd, TestPoint:TestPoint_Pad_D1.0mm, symbol Connector:TestPoint_Small
- C1: footprint (none) -> Capacitor_SMD:C_0402_1005Metric
- C2, C3, C4: footprint (none) -> Capacitor_SMD:C_0805_2012Metric
- C6: footprint Capacitor_SMD:C_0603_1608Metric -> Capacitor_SMD:C_0402_1005Metric
- D1: value Zener 400mW 3,3V -> D_Zener_Small; footprint (none) -> DIY:SOD323_bättre (2022_12_20 17_46_41 UTC)
- J1: footprint (none) -> Connector_PinHeader_2.54mm:PinHeader_1x03_P2.54mm_Vertical
- Q2, Q3, Q5, Q6, Q8, Q9: footprint (none) -> Package_DFN_QFN:DFN-8-1EP_3x3mm_P0.5mm_EP1.65x2.38mm
- R1, R10, R11, R12, R13, R14, R15, R16, R17, R18, R19, R2, R20, R3, R4, R5, R6, R7, R8, R9: footprint (none) -> Resistor_SMD:R_0402_1005Metric
- R21: value 220 -> 330; footprint (none) -> Resistor_SMD:R_0402_1005Metric
- TP5: value Test -> gnd; footprint (none) -> TestPoint:TestPoint_Pad_3.0x3.0mm
- TP6: value Test -> c2d; footprint (none) -> TestPoint:TestPoint_Pad_D1.0mm
- TP7: value Test -> p0,4; footprint (none) -> TestPoint:TestPoint_Pad_D1.0mm
Connections:
- net +3.3V: now also R11.1, R21.1, R5.1, R8.1, TP10.1; no longer R21.2
- net +5V: now also R21.2, J2.2 (Pin_2); no longer R21.1
- net GND: now also C9.2, J2.3 (Pin_3), TP2.1, TP9.1
- net VCC: now also C9.1, FB1.1, TP1.1, TP4.1; no longer C5.2, R11.1, R5.1, R8.1, U2.1 (VIN), U2.3 (ON/~{OFF})
- net at R1.2, U1.5 (RSTb/C2CK): now also TP8.1
- net at J1.1 (Pin_1), R2.1: now also J2.1 (Pin_1)
- net at R2.2, U1.17 (P0.5): now also TP3.1
- new net: C5.2, FB1.2, U2.1 (VIN), U2.3 (ON/~{OFF})
Other:
- moved on the sheet: C1, C2, C3, C4, C5, C6, J1, Q1, Q2, Q3, Q4, Q5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
