File: single/single_esc.kicad_sch (KiCad schematic)
At the start: 37 parts, among them T201 BC847, T202 BC847, T203 BC847, U201 EFM8BB10

Commit message: ok now it works in 7. i think
Parts:
- added Q1: BC847, Package_TO_SOT_SMD:SOT-23, symbol Transistor_BJT:BC847
- renumbered C201 to C501, C202 to C502, OUT_A201 to OUT_A501, OUT_B201 to OUT_B501, OUT_C201 to OUT_C501, R201 to R501, R202 to R502, R203 to R503, R204 to R504, R205 to R505, R206 to R506, R207 to R507, TP202 to TP502, U201 to U501
Changed lines of the file:
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@@
     (stroke (width 0) (type default))
   )
-  (label "Ac_0" (at 139.065 86.36 0) (fields_autoplaced)
+  (label "Ac_0" (at 139.065 86.36 0)
     (effects (font (size 1.524 1.524)) (justify left bottom))
   )
-  (label "Bp_0" (at 179.07 133.985 0) (fields_autoplaced)
+  (label "Bp_0" (at 179.07 133.985 0)
     (effects (font (size 1.524 1.524)) (justify left bottom))
   )
-  (label "Cc_0" (at 104.775 149.86 0) (fields_autoplaced)
+  (label "Cc_0" (at 104.775 149.86 0)
     (effects (font (size 1.524 1.524)) (justify left bottom))
   )
-  (label "PHASE_B_0" (at 215.9 104.14 0) (fields_autoplaced)
+  (label "PHASE_B_0" (at 215.9 104.14 0)
     (effects (font (size 1.524 1.524)) (justify left bottom))
   )
-  (label "Cp_0" (at 179.07 133.985 0) (fields_autoplaced)
+  (label "Cp_0" (at 179.07 133.985 0)
     (effects (font (size 1.524 1.524)) (justify left bottom))
   )
-  (label "RC_IN_0" (at 46.355 55.245 0) (fields_autoplaced)
+  (label "RC_IN_0" (at 46.355 55.245 0)
     (effects (font (size 1.524 1.524)) (justify left bottom))
   )
-  (label "Bp_0" (at 179.07 102.235 0) (fields_autoplaced)
+  (label "Bp_0" (at 179.07 102.235 0)
     (effects (font (size 1.524 1.524)) (justify left bottom))
   )
-  (label "Ap_0" (at 139.065 83.82 0) (fields_autoplaced)
+  (label "Ap_0" (at 139.065 83.82 0)
     (effects (font (size 1.524 1.524)) (justify left bottom))
   )
-  (label "C2D_0" (at 45.72 100.33 0) (fields_autoplaced)
+  (label "C2D_0" (at 45.72 100.33 0)
     (effects (font (size 1.524 1.524)) (justify left bottom))
   )
-  (label "Bc_0" (at 141.605 118.11 0) (fields_autoplaced)
+  (label "Bc_0" (at 141.605 118.11 0)
     (effects (font (size 1.524 1.524)) (justify left bottom))
   )
-  (label "PHASE_C_0" (at 214.63 137.795 0) (fields_autoplaced)
+  (label "PHASE_C_0" (at 214.63 137.795 0)
     (effects (font (size 1.524 1.524)) (justify left bottom))
   )
-  (label "C2CK_0" (at 46.355 88.9 0) (fields_autoplaced)
+  (label "C2CK_0" (at 46.355 88.9 0)
     (effects (font (size 1.524 1.524)) (justify left bottom))
   )
-  (label "PHASE_A_0" (at 215.9 72.39 0) (fields_autoplaced)
+  (label "PHASE_A_0" (at 215.9 72.39 0)
     (effects (font (size 1.524 1.524)) (justify left bottom))
   )
-  (hierarchical_label "RC_IN" (shape input) (at 45.72 55.245 180) (fields_autoplaced)
+  (hierarchical_label "RC_IN" (shape input) (at 45.72 55.245 180)
     (effects (font (size 1.524 1.524)) (justify right))
   )
-  (hierarchical_label "3V3" (shape input) (at 34.29 84.455 180) (fields_autoplaced)
+  (hierarchical_label "3V3" (shape input) (at 34.29 84.455 180)
     (effects (font (size 1.524 1.524)) (justify right))
   )
-  (hierarchical_label "GND" (shape input) (at 33.02 65.405 180) (fields_autoplaced)
+  (hierarchical_label "GND" (shape input) (at 33.02 65.405 180)
     (effects (font (size 1.524 1.524)) (justify right))
   )
-  (hierarchical_label "VCC" (shape input) (at 34.29 79.375 180) (fields_autoplaced)
+  (hierarchical_label "VCC" (shape input) (at 34.29 79.375 180)
     (effects (font (size 1.524 1.524)) (justify right))
   )
   (symbol (lib_id "custom:EFM8BB10") (at 88.9 91.44 0) (unit 1)
     (in_bom yes) (on_board yes) (dnp no)
-    (property "Reference" "U201" (at 99.06 85.09 0)
+    (property "Reference" "U501" (at 99.06 85.09 0)
       (effects (font (size 1.524 1.524)))
     )
@@
   (symbol (lib_id "custom:TP") (at 36.83 100.33 180) (unit 1)
     (in_bom yes) (on_board yes) (dnp no)
-    (property "Reference" "TP202" (at 33.02 100.33 0)
+    (property "Reference" "TP502" (at 33.02 100.33 0)
       (effects (font (size 1.524 1.524)))
     )
@@
   (symbol (lib_id "custom:CUSTOM_R") (at 233.68 55.245 0) (unit 1)
     (in_bom yes) (on_board yes) (dnp no)
-    (property "Reference" "R203" (at 235.712 55.245 90)
+    (property "Reference" "R503" (at 235.712 55.245 90)
       (effects (font (size 1.016 1.016)))
     )
@@
   (symbol (lib_id "custom:CUSTOM_R") (at 238.76 55.245 0) (unit 1)
     (in_bom yes) (on_board yes) (dnp no)
-    (property "Reference" "R205" (at 240.792 55.245 90)
+    (property "Reference" "R505" (at 240.792 55.245 90)
       (effects (font (size 1.016 1.016)))
     )
@@
   (symbol (lib_id "custom:CUSTOM_R") (at 243.84 55.245 0) (unit 1)
     (in_bom yes) (on_board yes) (dnp no)
-    (property "Reference" "R207" (at 245.872 55.245 90)
+    (property "Reference" "R507" (at 245.872 55.245 90)
       (effects (font (size 1.016 1.016)))
     )
@@
   (symbol (lib_id "custom:CUSTOM_R") (at 233.68 36.195 0) (unit 1)
     (in_bom yes) (on_board yes) (dnp no)
-    (property "Reference" "R202" (at 235.712 36.195 90)
+    (property "Reference" "R502" (at 235.712 36.195 90)
       (effects (font (size 1.016 1.016)))
     )
@@
   (symbol (lib_id "custom:CUSTOM_R") (at 238.76 36.195 0) (unit 1)
     (in_bom yes) (on_board yes) (dnp no)
-    (property "Reference" "R204" (at 240.792 36.195 90)
+    (property "Reference" "R504" (at 240.792 36.195 90)
       (effects (font (size 1.016 1.016)))
     )
@@
   (symbol (lib_id "custom:CUSTOM_R") (at 243.84 36.195 0) (unit 1)
     (in_bom yes) (on_board yes) (dnp no)
-    (property "Reference" "R206" (at 245.872 36.195 90)
+    (property "Reference" "R506" (at 245.872 36.195 90)
       (effects (font (size 1.016 1.016)))
     )
@@
   (symbol (lib_id "custom:TP") (at 254 72.39 0) (unit 1)
     (in_bom yes) (on_board yes) (dnp no)
-    (property "Reference" "OUT_A201" (at 257.81 72.39 0)
+    (property "Reference" "OUT_A501" (at 257.81 72.39 0)
       (effects (font (size 1.524 1.524)))
     )
@@
   (symbol (lib_id "custom:TP") (at 254 104.14 0) (unit 1)
     (in_bom yes) (on_board yes) (dnp no)
-    (property "Reference" "OUT_B201" (at 257.81 104.14 0)
+    (property "Reference" "OUT_B501" (at 257.81 104.14 0)
       (effects (font (size 1.524 1.524)))
     )
@@
   (symbol (lib_id "custom:TP") (at 254 137.795 0) (unit 1)
     (in_bom yes) (on_board yes) (dnp no)
-    (property "Reference" "OUT_C201" (at 257.81 137.795 0)
+    (property "Reference" "OUT_C501" (at 257.81 137.795 0)
       (effects (font (size 1.524 1.524)))
     )
@@
   (symbol (lib_id "custom:CUSTOM_C") (at 40.64 71.755 0) (unit 1)
     (in_bom yes) (on_board yes) (dnp no)
-    (property "Reference" "C201" (at 40.64 69.215 0)
+    (property "Reference" "C501" (at 40.64 69.215 0)
       (effects (font (size 1.016 1.016)) (justify left))
     )
@@
   (symbol (lib_id "custom:CUSTOM_C") (at 45.72 71.755 0) (unit 1)
     (in_bom yes) (on_board yes) (dnp no)
-    (property "Reference" "C202" (at 45.72 69.215 0)
+    (property "Reference" "C502" (at 45.72 69.215 0)
       (effects (font (size 1.016 1.016)) (justify left))
     )
@@
   (symbol (lib_id "custom:CUSTOM_R") (at 42.545 88.9 90) (unit 1)
     (in_bom yes) (on_board yes) (dnp no)
-    (property "Reference" "R201" (at 42.545 86.868 90)
+    (property "Reference" "R501" (at 42.545 86.868 90)
       (effects (font (size 1.016 1.016)))
     )
@@
   (symbol (lib_id "power:VCC") (at 154.94 75.565 0) (unit 1)
     (in_bom yes) (on_board yes) (dnp no)
-    (property "Reference" "#PWR055" (at 154.94 73.025 0)
+    (property "Reference" "#PWR010" (at 154.94 73.025 0)
       (effects (font (size 0.762 0.762)) hide)
     )
@@
   (symbol (lib_id "power:GND") (at 161.29 97.79 0) (unit 1)
     (in_bom yes) (on_board yes) (dnp no)
-    (property "Reference" "#PWR056" (at 161.29 97.79 0)
+    (property "Reference" "#PWR011" (at 161.29 97.79 0)
       (effects (font (size 0.762 0.762)) hide)
     )
@@
   (symbol (lib_id "power:GND") (at 161.29 129.54 0) (unit 1)
     (in_bom yes) (on_board yes) (dnp no)
-    (property "Reference" "#PWR057" (at 161.29 129.54 0)
+    (property "Reference" "#PWR012" (at 161.29 129.54 0)
       (effects (font (size 0.762 0.762)) hide)
     )
@@
   (symbol (lib_id "power:VCC") (at 152.4 107.315 0) (unit 1)
     (in_bom yes) (on_board yes) (dnp no)
-    (property "Reference" "#PWR058" (at 152.4 104.775 0)
+    (property "Reference" "#PWR013" (at 152.4 104.775 0)
       (effects (font (size 0.762 0.762)) hide)
     )
@@
   (symbol (lib_id "power:GND") (at 161.29 161.925 0) (unit 1)
     (in_bom yes) (on_board yes) (dnp no)
-    (property "Reference" "#PWR059" (at 161.29 161.925 0)
+    (property "Reference" "#PWR014" (at 161.29 161.925 0)
       (effects (font (size 0.762 0.762)) hide)
     )
@@
   (symbol (lib_id "power:VCC") (at 152.4 139.7 0) (unit 1)
     (in_bom yes) (on_board yes) (dnp no)
-    (property "Reference" "#PWR060" (at 152.4 137.16 0)
+    (property "Reference" "#PWR015" (at 152.4 137.16 0)
       (effects (font (size 0.762 0.762)) hide)
     )
@@
   (symbol (lib_id "power:GND") (at 273.685 52.705 0) (unit 1)
     (in_bom yes) (on_board yes) (dnp no)
-    (property "Reference" "#PWR054" (at 273.685 52.705 0)
+    (property "Reference" "#PWR09" (at 273.685 52.705 0)
       (effects (font (size 0.762 0.762)) hide)
     )
@@
         )
       )
+    )
+  )
+  (symbol (lib_id "Transistor_BJT:BC847") (at 139.7 101.6 0) (unit 1)
+    (in_bom yes) (on_board yes) (dnp no) (fields_autoplaced)
+    (property "Reference" "Q1" (at 144.78 100.33 0)
+      (effects (font (size 1.27 1.27)) (justify left))
+    )
+    (property "Value" "BC847" (at 144.78 102.87 0)
+      (effects (font (size 1.27 1.27)) (justify left))
+    )
+    (property "Footprint" "Package_TO_SOT_SMD:SOT-23" (at 144.78 103.505 0)
+      (effects (font (size 1.27 1.27) italic) (justify left) hide)
+    )
+    (property "Datasheet" "http://www.infineon.com/dgdl/Infineon-BC847SERIES_BC848SERIES_BC849SERIES_BC850SERIES-DS-v01_01-en.pdf?fileId=db3a304314dca389011541d4630a1657" (at 139.7 101.6 0)
+      (effects (font (size 1.27 1.27)) (justify left) hide)
+    )
+    (pin "1")
+    (pin "2")
+    (pin "3")
+    (instances
+      (project "single_esc"
+        (path "/f22a7b6c-63bc-4e09-8e0c-74ca594f4985"
+          (reference "Q1") (unit 1)
+        )
+      )
